Commit message: Camera TF fixed.

File: environment/urdf/objects/slab1.urdf (robot description, URDF)
Before this commit: robot slab, 1 links, 0 joints
Links:
- link slab: geometry collision box size=0.02 0.35 0.1; visual box size=0.02 0.35 0.1

Commit message: fix grasp orientation bug.

File: environment/urdf/objects/slab1.urdf (robot description, URDF)
Before this commit: robot slab, 1 links, 0 joints
Links:
- link slab: mass 0.1 -> 0.3

File: objects/ycb_objects/YcbTomatoSoupCan/model.urdf (robot description, URDF)
Before this commit: robot model.urdf, 1 links, 0 joints
Links:
- link baseLink: mass .1 -> .2; geometry collision mesh filename=collision_vhacd.obj scale=0.5 0.5 0.5; visual mesh filename=textured_simple_reoriented.obj scale=0.5 0.5 0.5

Commit message: Add geraspDetection demo

File: environment/urdf/objects/slab1.urdf (robot description, URDF)
Before this commit: robot slab, 1 links, 0 joints
Links:
- link slab: geometry collision box size=0.02 0.35 0.15; visual box size=0.02 0.35 0.15

Commit message: some other demo scripts.

File: environment/urdf/objects/slab1.urdf (robot description, URDF)
Before this commit: robot slab, 1 links, 0 joints
Links:
- link slab: geometry collision box size=0.02 0.35 0.05; visual box size=0.02 0.35 0.05

File: environment/urdf/objects/slab2.urdf (robot description, URDF)
Before this commit: robot slab2, 1 links, 0 joints
Links:
- link slab2: geometry collision box size=0.02 0.35 0.15; visual box size=0.02 0.35 0.15
