Commit message: Initial branch for Yucheng

File: objects/ycb_objects/YcbTube/model.urdf (robot description, URDF)
Before this commit: robot model.urdf, 1 links, 0 joints
Links:
- removed link baseLink
- added link base_link, mass 0.025; collision mesh filename=tube.obj; visual mesh filename=tube.obj
